File: astabile-kippstufe.sch (KiCad schematic (older format))
At the start: 16 parts, among them X1 +UB, X2 0V

Commit message: wires modified and mounting holes
Parts:
- added H1, H2, H3, H4: MountingHole, MountingHole:MountingHole_3.2mm_M3, symbol Mechanical:MountingHole
Changed lines of the file:
@@
+	1    0    0    -1
+$EndComp
+$Comp
+L Mechanical:MountingHole H1
+U 1 1 5EF0A1B5
+P 12200 5600
+F 0 "H1" H 12300 5646 50  0000 L CNN
+F 1 "MountingHole" H 12300 5555 50  0000 L CNN
+F 2 "MountingHole:MountingHole_3.2mm_M3" H 12200 5600 50  0001 C CNN
+F 3 "~" H 12200 5600 50  0001 C CNN
+	1    12200 5600
+	1    0    0    -1
+$EndComp
+$Comp
+L Mechanical:MountingHole H2
+U 1 1 5EF0D522
+P 12200 5850
+F 0 "H2" H 12300 5896 50  0000 L CNN
+F 1 "MountingHole" H 12300 5805 50  0000 L CNN
+F 2 "MountingHole:MountingHole_3.2mm_M3" H 12200 5850 50  0001 C CNN
+F 3 "~" H 12200 5850 50  0001 C CNN
+	1    12200 5850
+	1    0    0    -1
+$EndComp
+$Comp
+L Mechanical:MountingHole H3
+U 1 1 5EF0D6C0
+P 12200 6100
+F 0 "H3" H 12300 6146 50  0000 L CNN
+F 1 "MountingHole" H 12300 6055 50  0000 L CNN
+F 2 "MountingHole:MountingHole_3.2mm_M3" H 12200 6100 50  0001 C CNN
+F 3 "~" H 12200 6100 50  0001 C CNN
+	1    12200 6100
+	1    0    0    -1
+$EndComp
+$Comp
+L Mechanical:MountingHole H4
+U 1 1 5EF0D8E4
+P 12200 6350
+F 0 "H4" H 12300 6396 50  0000 L CNN
+F 1 "MountingHole" H 12300 6305 50  0000 L CNN
+F 2 "MountingHole:MountingHole_3.2mm_M3" H 12200 6350 50  0001 C CNN
+F 3 "~" H 12200 6350 50  0001 C CNN
+	1    12200 6350
 	1    0    0    -1
 $EndComp
